File: Eagle_files/Final Project Designs.sch (EAGLE design)
At the start: 29 parts, among them M1 30V, U1 LM3488MMX/NOPB

Commit message: Modified 14 pin header to include screw hole layout for lcd
Parts:
- removed CBP: 100nF, AcceleratedDesigns_Lib:GRM155R61A104KA01DGRM155R61A104KA01D
- removed CCOMP: 82nF, AcceleratedDesigns_Lib:GRM155R61A823KA01DGRM155R61A823KA01D
- removed CCOMP2: 5.1nF, AcceleratedDesigns_Lib:GRM2195C1H512JA01DGRM2195C1H512JA01D
- removed COUT_1, COUT_2: 100uF, AcceleratedDesigns_Lib:GRM31CR60J107ME39LGRM31CR60J107ME39L
- removed CRAMP: 1.2nF, AcceleratedDesigns_Lib:CL21C122JBFNNWECL21C122JBFNNWE
- removed CSEP: 2.2uF, AcceleratedDesigns_Lib:GRM21BR71A225KA01LGRM21BR71A225KA01L
- removed D1: 500mV, AcceleratedDesigns_Lib:B220-13-FB220-13-F
- removed E$1, E$2: MICRO-USB-ZX62R-B-5P, con-hirose:MICRO-USB-ZX62R-B-5P
- removed GND100: WB_GND, AcceleratedDesigns_Lib:WB_GNDWB_GND
- removed LIN: 12uH, AcceleratedDesigns_Lib:NPI75C120MTRFNPI75C120MTRF
- removed LOUT: 33uH, AcceleratedDesigns_Lib:SRN8040-330MSRN8040-330M
- removed M1: 30V, AcceleratedDesigns_Lib:CSD17308Q3CSD17308Q3
- removed RBP: 20, AcceleratedDesigns_Lib:CRCW040220R0FKEDCRCW040220R0FKED
- removed RCOMP: 1.18k, AcceleratedDesigns_Lib:CRCW04021K18FKEDCRCW04021K18FKED
- removed RFADJ: 69.8k, AcceleratedDesigns_Lib:CRCW040269K8FKEDCRCW040269K8FKED
- removed RFB1: 10k, AcceleratedDesigns_Lib:CRCW040210K0FKEDCRCW040210K0FKED
- removed RFB2: 16.2k, AcceleratedDesigns_Lib:CRCW040216K2FKEDCRCW040216K2FKED
- removed RRAMP: 100, AcceleratedDesigns_Lib:CRCW0402100RFKEDCRCW0402100RFKED
- removed RSENSE: 33m, AcceleratedDesigns_Lib:ERJ-L14KF33MUERJ-L14KF33MU
- added COUT, COUTX: 10uF, AcceleratedDesigns_Lib:CL10A106MQ8NNNCCL10A106MQ8NNNC
- added CSS: 1nF, AcceleratedDesigns_Lib:GRM155R61A102KA01DGRM155R61A102KA01D
- added L1: 1.5uH, AcceleratedDesigns_Lib:LQM2HPN1R5MG0LLQM2HPN1R5MG0L
- added RPG: 100k, AcceleratedDesigns_Lib:CRCW0603100KFKEACRCW0603100KFKEA
- CIN: value 4.7uF -> 10uF; device AcceleratedDesigns_Lib:10TPU4R7MSI10TPU4R7MSI -> AcceleratedDesigns_Lib:LMK107BBJ106MAHTLMK107BBJ106MAHT
- U1: value LM3488MMX/NOPB -> TPS63051YFFR; device AcceleratedDesigns_Lib:LM3488MMX/NOPBLM3488MMX/NOPB -> AcceleratedDesigns_Lib:TPS63051YFFRTPS63051YFFR
Connections:
- removed net 1: RFADJ.2@2, U1.FA/SYNC/SD@7
- removed net 10: CSEP.2@2, LIN.1@1, M1.DRAIN@1, M1.DRAIN@2, M1.DRAIN@3, M1.DRAIN@4, M1.DRAIN@5
- removed net 11: M1.GATE@6, U1.DR@6
- removed net 12: RRAMP.1@1, U1.ISEN@1
- removed net 13: CCOMP.1@1, RCOMP.2@2
- removed net 7: CBP.1@1, RBP.2@2, U1.VIN@8
- removed net 9: M1.SOURCE@7, M1.SOURCE@8, M1.SOURCE@9, RRAMP.2@2, RSENSE.1@1
- net 0: now also CIN.2@2, COUT.2@2, COUTX.2@2, CSS.2@2, U1.GND@4, U1.PFM_PWM@8; no longer CBP.2@2, CCOMP.2@2, CCOMP2.2@2, CIN.-@2, COUT_1.2@2, COUT_2.2@2, CRAMP.2@2, GND100.1@1, LOUT.2@2, RFADJ.1@1, RFB1.2@2, RSENSE.2@2, U1.AGND@4, U1.PGND@5
- net 2: now also CIN.1@1, U1.EN@3, U1.ILIM0@5, U1.ILIM1@6, U1.VIN@2, VIN.+@1; no longer COUT_1.1@1, COUT_2.1@1, D1.K@2, IOUT.+@1, RFB2.1@1
- net 3: now also CSS.1@1, U1.SS@12; no longer CIN.+@1, LIN.2@2, RBP.1@1, VIN.+@1
- net 4: now also COUT.1@1, COUTX.1@1, IOUT.+@1, RPG.1@1, U1.FB@11, U1.VOUT@10; no longer CCOMP2.1@1, RCOMP.1@1, U1.COMP@2
- net 5: now also L1.1@1, U1.L1@1; no longer CSEP.1@1, D1.A@1, LOUT.1@1
- net 6: now also L1.2@2, U1.L2@7; no longer CRAMP.1@1
- net 8: now also RPG.2@2, U1.PG@9; no longer RFB1.1@1, RFB2.2@2, U1.FB@3
Other:
- moved on the sheet: CIN, IOUT, VIN

Commit message: building the schematic
Parts:
- removed CIN: 10uF, AcceleratedDesigns_Lib:LMK107BBJ106MAHTLMK107BBJ106MAHT
- removed COUT, COUTX: 10uF, AcceleratedDesigns_Lib:CL10A106MQ8NNNCCL10A106MQ8NNNC
- removed CSS: 1nF, AcceleratedDesigns_Lib:GRM155R61A102KA01DGRM155R61A102KA01D
- removed E$3: (no value), con-berg:PN87520
- removed GND: WB_GND, AcceleratedDesigns_Lib:WB_GNDWB_GND
- removed IOUT: WB_CURRENT_LOAD, AcceleratedDesigns_Lib:WB_CURRENT_LOADWB_CURRENT_LOAD
- removed L1: 1.5uH, AcceleratedDesigns_Lib:LQM2HPN1R5MG0LLQM2HPN1R5MG0L
- removed RPG: 100k, AcceleratedDesigns_Lib:CRCW0603100KFKEACRCW0603100KFKEA
- removed U1: TPS63051YFFR, AcceleratedDesigns_Lib:TPS63051YFFRTPS63051YFFR
- removed VIN: WB_BATTERY, AcceleratedDesigns_Lib:WB_BATTERYWB_BATTERY
- added IC1: ATXMEGA32AA, Tft_lcd_header:ATXMEGA32AA
- added J1, J2: USB-MICROB", SparkFun-Connectors:USB-MICROB"
- added SW1, SW2: (no value), buttons:10-XX-4.5SMD
- added X1: (no value), con-berg:PN87520
Connections:
- removed net 0: CIN.2@2, COUT.2@2, COUTX.2@2, CSS.2@2, GND.1@1, IOUT.-@2, U1.GND@4, U1.PFM_PWM@8, VIN.-@2
- removed net 2: CIN.1@1, U1.EN@3, U1.ILIM0@5, U1.ILIM1@6, U1.VIN@2, VIN.+@1
- removed net 3: CSS.1@1, U1.SS@12
- removed net 4: COUT.1@1, COUTX.1@1, IOUT.+@1, RPG.1@1, U1.FB@11, U1.VOUT@10
- removed net 5: L1.1@1, U1.L1@1
- removed net 6: L1.2@2, U1.L2@7
- removed net 8: RPG.2@2, U1.PG@9
- new net +3V3: IC1.AVCC, IC1.VCC, SV1.LED, SV1.VCC, SW1.P1, SW2.P1, U$1.VCC
- new net GND: IC1.GND, SV1.GND
- new net N$1: IC1.(MOSI)PC7, SV1.MOSI
- new net N$10: IC1.(RXD)PD0, SW1.S1
- new net N$11: U$1.GND
- new net N$12: J1.VBUS
- new net N$13: X1.1
- new net N$2: SV1.SCK
- new net N$3: IC1.(MISO)PC6, SV1.MISO
- new net N$4: IC1.(SCL)PC1, U$1.SCL
- new net N$5: U$1.SDA
- new net N$6: X1.4
- new net N$7: J1.D+, X1.2
- new net N$8: J1.D-
- new net N$9: IC1.(TXD)PD1, SW2.S1
