File: Eagle_files/Final Project Designs_v1.sch (EAGLE design)
At the start: 8 parts, among them IC1 ATXMEGA32AA, J1 USB-MICROB"

Commit message: updated designs
Parts:
- added U$3, U$4: BANANA_PLUG, Tft_lcd_header:BANANA_PLUG
- added U$5: FUSE_SMT, fuse_smt:FUSE_SMT
Connections:
- removed net N$12: J1.VBUS, U$2.I_IN
- removed net N$13: U$2.I_OUT, X1.1
- new net B$1: J1.VBUS, U$2.I_IN, U$4.BP
- new net B$2: U$3.BP, U$5.P$2
- new net N$16: U$2.I_OUT, U$5.P$1
Changed lines of the file:
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@@
 <part name="SW2" library="buttons" deviceset="10-XX" device="-4.5SMD"/>
 <part name="U$2" library="Tft_lcd_header" deviceset="RESISTOR_4PIN" device=""/>
+<part name="U$3" library="Tft_lcd_header" deviceset="BANANA_PLUG" device=""/>
+<part name="U$4" library="Tft_lcd_header" deviceset="BANANA_PLUG" device=""/>
+<part name="U$5" library="fuse_smt" deviceset="FUSE_SMT" device=""/>
 </parts>
 <sheets>
@@
 <instance part="SW2" gate="1" x="45.72" y="83.82"/>
 <instance part="U$2" gate="G$1" x="119.38" y="66.04" smashed="yes"/>
+<instance part="U$3" gate="G$1" x="134.62" y="25.4"/>
+<instance part="U$4" gate="G$1" x="134.62" y="106.68"/>
+<instance part="U$5" gate="G$1" x="119.38" y="38.1" rot="R90"/>
 </instances>
 <busses>
@@
 <wire x1="93.98" y1="43.18" x2="109.22" y2="43.18" width="0.1524" layer="91"/>
 <wire x1="109.22" y1="43.18" x2="109.22" y2="50.8" width="0.1524" layer="91"/>
+<junction x="93.98" y="43.18"/>
 </segment>
 <segment>
@@
 <pinref part="SW1" gate="1" pin="P1"/>
 <pinref part="SW2" gate="1" pin="P1"/>
+<junction x="38.1" y="93.98"/>
 </segment>
 </net>
@@
 </segment>
 </net>
-<net name="N$12" class="0">
+<net name="B$1" class="0">
 <segment>
 <pinref part="J1" gate="G$1" pin="VBUS"/>
@@
 <wire x1="119.38" y1="91.44" x2="119.38" y2="81.28" width="0.1524" layer="91"/>
 <pinref part="U$2" gate="G$1" pin="I_IN"/>
-</segment>
-</net>
-<net name="N$13" class="0">
-<segment>
-<pinref part="X1" gate="G$1" pin="1"/>
-<wire x1="134.62" y1="40.64" x2="119.38" y2="40.64" width="0.1524" layer="91"/>
-<wire x1="119.38" y1="40.64" x2="119.38" y2="53.34" width="0.1524" layer="91"/>
-<pinref part="U$2" gate="G$1" pin="I_OUT"/>
-<wire x1="119.38" y1="53.34" x2="119.38" y2="55.88" width="0.1524" layer="91"/>
-<junction x="119.38" y="53.34"/>
+<wire x1="119.38" y1="91.44" x2="119.38" y2="106.68" width="0.1524" layer="91"/>
+<junction x="119.38" y="91.44"/>
+<pinref part="U$4" gate="G$1" pin="BP"/>
+<wire x1="134.62" y1="106.68" x2="119.38" y2="106.68" width="0.1524" layer="91"/>
 </segment>
 </net>
@@
 </segment>
 </net>
+<net name="N$16" class="0">
+<segment>
+<pinref part="U$2" gate="G$1" pin="I_OUT"/>
+<wire x1="119.38" y1="48.26" x2="119.38" y2="53.34" width="0.1524" layer="91"/>
+<pinref part="U$5" gate="G$1" pin="P$1"/>
+</segment>
+</net>
+<net name="B$2" class="0">
+<segment>
+<wire x1="119.38" y1="22.86" x2="132.08" y2="22.86" width="0.1524" layer="91"/>
+<wire x1="132.08" y1="22.86" x2="132.08" y2="25.4" width="0.1524" layer="91"/>
+<wire x1="132.08" y1="25.4" x2="132.08" y2="40.64" width="0.1524" layer="91"/>
+<wire x1="132.08" y1="40.64" x2="137.16" y2="40.64" width="0.1524" layer="91"/>
+<wire x1="119.38" y1="25.4" x2="119.38" y2="22.86" width="0.1524" layer="91"/>
+<pinref part="U$5" gate="G$1" pin="P$2"/>
+<pinref part="U$3" gate="G$1" pin="BP"/>
+<wire x1="134.62" y1="25.4" x2="132.08" y2="25.4" width="0.1524" layer="91"/>
+<junction x="132.08" y="25.4"/>
+</segment>
+</net>
