File: Eagle_files/Final Project Designs_v1.sch (EAGLE design)
At the start: 20 parts, among them CON1 header, CON2 4PIN_GROVE_CONNECTORUNIVERSAL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, U2 ATXMEGA32AA, X1 USB-MICROB", X4 JTAG, X5 BANANA_PLUG, X6 BANANA_PLUG

Commit message: finished the schematic and board designs
Parts:
- added CIN: LMK212BJ106KG-T, sps:LMK212BJ106KG-T
- added COUT_1, COUT_2: LMK212BJ226MG-T, sps:LMK212BJ226MG-T
- added GND-, VIN+: TP-1502, sps:TP-1502
- added L1: LQM21PN1R5MC0D, sps:LQM21PN1R5MC0D
- added RFBB: CRCW0402178KFKED, sps:CRCW0402178KFKED
- added RFBT: CRCW04021M00FKED, sps:CRCW04021M00FKED
- added U1: TPS63000DRCR, sps:TPS63000DRCR
Connections:
- new net 2: L1.1, U1.L1
- new net 3V3: COUT_1.1, COUT_2.1, RFBT.1, U1.VOUT
- new net 4: L1.2, U1.L2
- new net N$31: RFBB.1, RFBT.2, U1.FB
- new net VIN: CIN.1, U1.EN, U1.PS_SYNC, U1.VIN, U1.VINA, VIN+.TP
- net GND: now also CIN.2, COUT_1.2, COUT_2.2, GND-.TP, RFBB.2, U1.GND, U1.PAD, U1.PGND
Other:
- note added: "1.5uh"
- note added: "10uf"
- note added: "178k"
- note added: "1M"
- note added: "22uf"
Changed lines of the file:
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@@
 <part name="GND5" library="supply1" deviceset="GND" device=""/>
 <part name="GND6" library="supply1" deviceset="GND" device=""/>
+<part name="VIN+" library="sps" deviceset="TP-1502" device=""/>
+<part name="GND-" library="sps" deviceset="TP-1502" device=""/>
+<part name="RFBT" library="sps" deviceset="CRCW04021M00FKED" device=""/>
+<part name="RFBB" library="sps" deviceset="CRCW0402178KFKED" device=""/>
+<part name="CIN" library="sps" deviceset="LMK212BJ106KG-T" device=""/>
+<part name="COUT_1" library="sps" deviceset="LMK212BJ226MG-T" device=""/>
+<part name="COUT_2" library="sps" deviceset="LMK212BJ226MG-T" device=""/>
+<part name="L1" library="sps" deviceset="LQM21PN1R5MC0D" device=""/>
+<part name="U1" library="sps" deviceset="TPS63000DRCR" device=""/>
+<part name="+3V7" library="supply1" deviceset="+3V3" device=""/>
+<part name="GND7" library="supply1" deviceset="GND" device=""/>
 </parts>
 <sheets>
@@
 <instance part="GND5" gate="1" x="50.8" y="88.9"/>
 <instance part="GND6" gate="1" x="50.8" y="101.6"/>
+<instance part="+3V7" gate="G$1" x="-35.56" y="101.6"/>
+<instance part="GND7" gate="1" x="-35.56" y="76.2"/>
 </instances>
 <busses>
@@
 <wire x1="93.98" y1="12.7" x2="93.98" y2="15.24" width="0.1524" layer="91"/>
 </segment>
+<segment>
+<wire x1="-45.72" y1="93.98" x2="-35.56" y2="93.98" width="0.1524" layer="91"/>
+<pinref part="+3V7" gate="G$1" pin="+3V3"/>
+<wire x1="-35.56" y1="99.06" x2="-35.56" y2="93.98" width="0.1524" layer="91"/>
+</segment>
 </net>
 <net name="GND" class="0">
@@
 <pinref part="GND6" gate="1" pin="GND"/>
 <wire x1="48.26" y1="104.14" x2="50.8" y2="104.14" width="0.1524" layer="91"/>
+</segment>
+<segment>
+<wire x1="-45.72" y1="83.82" x2="-35.56" y2="83.82" width="0.1524" layer="91"/>
+<pinref part="GND7" gate="1" pin="GND"/>
+<wire x1="-35.56" y1="83.82" x2="-35.56" y2="78.74" width="0.1524" layer="91"/>
 </segment>
 </net>
@@
 <sheet>
 <plain>
+<text x="20.32" y="33.02" size="1.778" layer="91">10uf</text>
+<text x="124.46" y="30.48" size="1.778" layer="91">22uf</text>
+<text x="66.04" y="86.36" size="1.778" layer="91">1.5uh</text>
+<text x="104.14" y="50.8" size="1.778" layer="91">1M</text>
+<text x="104.14" y="22.86" size="1.778" layer="91">178k</text>
 </plain>
 <instances>
+<instance part="VIN+" gate="A" x="-2.54" y="66.04" smashed="yes">
+<attribute name="NAME" x="-30.1244" y="75.1586" size="2.0828" layer="95" ratio="6" rot="SR0"/>
+</instance>
+<instance part="GND-" gate="A" x="-2.54" y="10.16" smashed="yes">
+<attribute name="NAME" x="-30.1244" y="19.2786" size="2.0828" layer="95" ratio="6" rot="SR0"/>
+</instance>
+<instance part="RFBT" gate="A" x="93.98" y="55.88" smashed="yes" rot="R90">
+<attribute name="NAME" x="89.3064" y="51.1556" size="2.0828" layer="95" ratio="6" rot="SR90"/>
+</instance>
+<instance part="RFBB" gate="A" x="93.98" y="27.94" smashed="yes" rot="R90">
+<attribute name="NAME" x="89.3064" y="23.2156" size="2.0828" layer="95" ratio="6" rot="SR90"/>
+</instance>
+<instance part="CIN" gate="A" x="12.7" y="43.18" smashed="yes" rot="R90">
+<attribute name="NAME" x="6.1214" y="38.4556" size="2.0828" layer="95" ratio="6" rot="SR90"/>
+</instance>
+<instance part="COUT_1" gate="A" x="116.84" y="43.18" smashed="yes" rot="R90">
+<attribute name="NAME" x="110.2614" y="38.4556" size="2.0828" layer="95" ratio="6" rot="SR90"/>
+</instance>
+<instance part="COUT_2" gate="A" x="134.62" y="43.18" smashed="yes" rot="R90">
+<attribute name="NAME" x="128.0414" y="38.4556" size="2.0828" layer="95" ratio="6" rot="SR90"/>
+</instance>
+<instance part="L1" gate="A" x="55.88" y="91.44" smashed="yes">
+<attribute name="NAME" x="51.1556" y="96.1136" size="2.0828" layer="95" ratio="6" rot="SR0"/>
+</instance>
+<instance part="U1" gate="A" x="55.88" y="55.88" smashed="yes">
+<attribute name="NAME" x="51.1556" y="57.3786" size="2.0828" layer="95" ratio="6" rot="SR0"/>
+</instance>
 </instances>
 <busses>
 </busses>
 <nets>
+<net name="VIN" class="0">
+<segment>
+<wire x1="30.48" y1="48.26" x2="30.48" y2="55.88" width="0" layer="91"/>
+<wire x1="30.48" y1="55.88" x2="30.48" y2="60.96" width="0" layer="91"/>
+<wire x1="30.48" y1="60.96" x2="30.48" y2="66.04" width="0" layer="91"/>
+<wire x1="35.56" y1="48.26" x2="30.48" y2="48.26" width="0" layer="91"/>
+<wire x1="35.56" y1="55.88" x2="30.48" y2="55.88" width="0" layer="91"/>
+<junction x="30.48" y="55.88"/>
+<wire x1="35.56" y1="60.96" x2="30.48" y2="60.96" width="0" layer="91"/>
+<junction x="30.48" y="60.96"/>
+<wire x1="-2.54" y1="66.04" x2="12.7" y2="66.04" width="0.1524" layer="91"/>
+<wire x1="12.7" y1="66.04" x2="30.48" y2="66.04" width="0.1524" layer="91"/>
+<wire x1="30.48" y1="66.04" x2="35.56" y2="66.04" width="0.1524" layer="91"/>
+<wire x1="12.7" y1="50.8" x2="12.7" y2="66.04" width="0.1524" layer="91"/>
+<junction x="12.7" y="66.04"/>
+<junction x="30.48" y="66.04"/>
+<pinref part="VIN+" gate="A" pin="TP"/>
+<pinref part="CIN" gate="A" pin="1"/>
+<pinref part="U1" gate="A" pin="VIN"/>
+<pinref part="U1" gate="A" pin="EN"/>
+<pinref part="U1" gate="A" pin="PS_SYNC"/>
+<pinref part="U1" gate="A" pin="VINA"/>
+</segment>
+</net>
+<net name="GND" class="0">
+<segment>
+<wire x1="12.7" y1="10.16" x2="78.74" y2="10.16" width="0" layer="91"/>
+<wire x1="78.74" y1="10.16" x2="93.98" y2="10.16" width="0" layer="91"/>
+<wire x1="93.98" y1="10.16" x2="116.84" y2="10.16" width="0" layer="91"/>
+<wire x1="116.84" y1="10.16" x2="157.48" y2="10.16" width="0" layer="91"/>
+<label x="132.08" y="5.08" size="1.778" layer="95"/>
+<wire x1="12.7" y1="35.56" x2="12.7" y2="10.16" width="0.1524" layer="91"/>
+<wire x1="116.84" y1="35.56" x2="134.62" y2="35.56" width="0" layer="91"/>
+<wire x1="116.84" y1="35.56" x2="116.84" y2="10.16" width="0" layer="91"/>
+<junction x="116.84" y="10.16"/>
+<wire x1="-2.54" y1="10.16" x2="12.7" y2="10.16" width="0.1524" layer="91"/>
+<wire x1="76.2" y1="45.72" x2="78.74" y2="45.72" width="0.1524" layer="91"/>
+<wire x1="78.74" y1="45.72" x2="78.74" y2="40.64" width="0.1524" layer="91"/>
+<wire x1="78.74" y1="40.64" x2="78.74" y2="38.1" width="0.1524" layer="91"/>
+<wire x1="78.74" y1="38.1" x2="78.74" y2="10.16" width="0.1524" layer="91"/>
+<wire x1="76.2" y1="40.64" x2="78.74" y2="40.64" width="0.1524" layer="91"/>
+<wire x1="76.2" y1="38.1" x2="78.74" y2="38.1" width="0.1524" layer="91"/>
+<junction x="78.74" y="40.64"/>
+<junction x="78.74" y="38.1"/>
+<junction x="78.74" y="10.16"/>
+<junction x="12.7" y="10.16"/>
+<pinref part="GND-" gate="A" pin="TP"/>
+<wire x1="93.98" y1="20.32" x2="93.98" y2="10.16" width="0.1524" layer="91"/>
+<junction x="93.98" y="10.16"/>
+<pinref part="CIN" gate="A" pin="2"/>
+<pinref part="U1" gate="A" pin="PGND"/>
+<pinref part="U1" gate="A" pin="GND"/>
+<pinref part="U1" gate="A" pin="PAD"/>
+<pinref part="RFBB" gate="A" pin="2"/>
+<pinref part="COUT_1" gate="A" pin="2"/>
+<junction x="116.84" y="35.56"/>
+<pinref part="COUT_2" gate="A" pin="2"/>
+</segment>
+</net>
+<net name="3V3" class="0">
+<segment>
+<wire x1="116.84" y1="50.8" x2="116.84" y2="66.04" width="0" layer="91"/>
+<wire x1="116.84" y1="50.8" x2="134.62" y2="50.8" width="0" layer="91"/>
+<label x="129.54" y="68.58" size="1.778" layer="95"/>
+<junction x="116.84" y="66.04"/>
+<wire x1="76.2" y1="66.04" x2="93.98" y2="66.04" width="0" layer="91"/>
+<wire x1="93.98" y1="66.04" x2="116.84" y2="66.04" width="0" layer="91"/>
+<wire x1="116.84" y1="66.04" x2="157.48" y2="66.04" width="0" layer="91"/>
+<wire x1="93.98" y1="63.5" x2="93.98" y2="66.04" width="0.1524" layer="91"/>
+<junction x="93.98" y="66.04"/>
+<pinref part="U1" gate="A" pin="VOUT"/>
+<pinref part="RFBT" gate="A" pin="1"/>
+<pinref part="COUT_1" gate="A" pin="1"/>
+<junction x="116.84" y="50.8"/>
+<pinref part="COUT_2" gate="A" pin="1"/>
+</segment>
+</net>
+<net name="2" class="0">
+<segment>
+<wire x1="35.56" y1="71.12" x2="30.48" y2="71.12" width="0.1524" layer="91"/>
+<wire x1="30.48" y1="71.12" x2="30.48" y2="91.44" width="0.1524" layer="91"/>
+<wire x1="48.26" y1="91.44" x2="30.48" y2="91.44" width="0.1524" layer="91"/>
+<pinref part="L1" gate="A" pin="1"/>
+<pinref part="U1" gate="A" pin="L1"/>
+</segment>
+</net>
+<net name="4" class="0">
+<segment>
+<wire x1="81.28" y1="91.44" x2="81.28" y2="71.12" width="0.1524" layer="91"/>
+<wire x1="81.28" y1="71.12" x2="76.2" y2="71.12" width="0.1524" layer="91"/>
+<wire x1="63.5" y1="91.44" x2="81.28" y2="91.44" width="0.1524" layer="91"/>
+<pinref part="L1" gate="A" pin="2"/>
+<pinref part="U1" gate="A" pin="L2"/>
+</segment>
+</net>
+<net name="N$31" class="0">
+<segment>
+<wire x1="76.2" y1="55.88" x2="83.82" y2="55.88" width="0.1524" layer="91"/>
+<wire x1="83.82" y1="55.88" x2="83.82" y2="43.18" width="0.1524" layer="91"/>
+<wire x1="83.82" y1="43.18" x2="93.98" y2="43.18" width="0.1524" layer="91"/>
+<wire x1="93.98" y1="48.26" x2="93.98" y2="43.18" width="0.1524" layer="91"/>
+<wire x1="93.98" y1="43.18" x2="93.98" y2="35.56" width="0.1524" layer="91"/>
+<junction x="93.98" y="43.18"/>
+<pinref part="U1" gate="A" pin="FB"/>
+<pinref part="RFBT" gate="A" pin="2"/>
+<pinref part="RFBB" gate="A" pin="1"/>
+</segment>
+</net>
 </nets>
 </sheet>

Commit message: finished everthing
Parts:
- removed GND-, VIN+: TP-1502, sps:TP-1502
- added U$1: BATTERY, Tft_lcd_header:BATTERY
Connections:
- net GND: now also U$1.GND; no longer GND-.TP
- net VIN: now also U$1.PWR; no longer VIN+.TP
Changed lines of the file:
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@@
 <part name="GND5" library="supply1" deviceset="GND" device=""/>
 <part name="GND6" library="supply1" deviceset="GND" device=""/>
-<part name="VIN+" library="sps" deviceset="TP-1502" device=""/>
-<part name="GND-" library="sps" deviceset="TP-1502" device=""/>
 <part name="RFBT" library="sps" deviceset="CRCW04021M00FKED" device=""/>
 <part name="RFBB" library="sps" deviceset="CRCW0402178KFKED" device=""/>
@@
 <part name="+3V7" library="supply1" deviceset="+3V3" device=""/>
 <part name="GND7" library="supply1" deviceset="GND" device=""/>
+<part name="U$1" library="Tft_lcd_header" deviceset="BATTERY" device=""/>
 </parts>
 <sheets>
@@
 </plain>
 <instances>
-<instance part="VIN+" gate="A" x="-2.54" y="66.04" smashed="yes">
-<attribute name="NAME" x="-30.1244" y="75.1586" size="2.0828" layer="95" ratio="6" rot="SR0"/>
-</instance>
-<instance part="GND-" gate="A" x="-2.54" y="10.16" smashed="yes">
-<attribute name="NAME" x="-30.1244" y="19.2786" size="2.0828" layer="95" ratio="6" rot="SR0"/>
-</instance>
 <instance part="RFBT" gate="A" x="93.98" y="55.88" smashed="yes" rot="R90">
 <attribute name="NAME" x="89.3064" y="51.1556" size="2.0828" layer="95" ratio="6" rot="SR90"/>
@@
 <attribute name="NAME" x="51.1556" y="57.3786" size="2.0828" layer="95" ratio="6" rot="SR0"/>
 </instance>
+<instance part="U$1" gate="G$1" x="-15.24" y="43.18"/>
 </instances>
 <busses>
@@
 <wire x1="35.56" y1="60.96" x2="30.48" y2="60.96" width="0" layer="91"/>
 <junction x="30.48" y="60.96"/>
-<wire x1="-2.54" y1="66.04" x2="12.7" y2="66.04" width="0.1524" layer="91"/>
+<wire x1="-15.24" y1="66.04" x2="12.7" y2="66.04" width="0.1524" layer="91"/>
 <wire x1="12.7" y1="66.04" x2="30.48" y2="66.04" width="0.1524" layer="91"/>
 <wire x1="30.48" y1="66.04" x2="35.56" y2="66.04" width="0.1524" layer="91"/>
@@
 <junction x="12.7" y="66.04"/>
 <junction x="30.48" y="66.04"/>
-<pinref part="VIN+" gate="A" pin="TP"/>
 <pinref part="CIN" gate="A" pin="1"/>
 <pinref part="U1" gate="A" pin="VIN"/>
@@
 <pinref part="U1" gate="A" pin="PS_SYNC"/>
 <pinref part="U1" gate="A" pin="VINA"/>
+<pinref part="U$1" gate="G$1" pin="PWR"/>
+<wire x1="-15.24" y1="58.42" x2="-15.24" y2="66.04" width="0.1524" layer="91"/>
 </segment>
 </net>
@@
 <wire x1="116.84" y1="35.56" x2="116.84" y2="10.16" width="0" layer="91"/>
 <junction x="116.84" y="10.16"/>
-<wire x1="-2.54" y1="10.16" x2="12.7" y2="10.16" width="0.1524" layer="91"/>
+<wire x1="-15.24" y1="10.16" x2="12.7" y2="10.16" width="0.1524" layer="91"/>
 <wire x1="76.2" y1="45.72" x2="78.74" y2="45.72" width="0.1524" layer="91"/>
 <wire x1="78.74" y1="45.72" x2="78.74" y2="40.64" width="0.1524" layer="91"/>
@@
 <junction x="78.74" y="10.16"/>
 <junction x="12.7" y="10.16"/>
-<pinref part="GND-" gate="A" pin="TP"/>
 <wire x1="93.98" y1="20.32" x2="93.98" y2="10.16" width="0.1524" layer="91"/>
 <junction x="93.98" y="10.16"/>
@@
 <junction x="116.84" y="35.56"/>
 <pinref part="COUT_2" gate="A" pin="2"/>
-</segment>
-</net>
+<pinref part="U$1" gate="G$1" pin="GND"/>
+<wire x1="-15.24" y1="25.4" x2="-15.24" y2="10.16" width="0.1524" layer="91"/>
+</segment>
+</net>
