File: Eagle_files/Final Project Designs_v1_copy.brd (EAGLE design)
At the start: 100 x 80 mm, 29 parts, among them CON1 header, CON2 4PIN_GROVE_CONNECTORUNIVERSAL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, U1 TPS63000DRCR, U2 ATXMEGA32AA, X1 USB-MICROB", X4 JTAG, X5 BANANA_PLUG, X6 BANANA_PLUG

Commit message: added few more files
Routing:
- net N$15: track 4.70 -> 3.55 mm
- net B$2: track 29.0 -> 30.1 mm
Changed lines of the file:
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@@
 <contactref element="R1" pad="I_OUT"/>
 <contactref element="X3" pad="1"/>
-<wire x1="16.9" y1="16.5" x2="12.4239" y2="15.123878125" width="4" layer="1"/>
+<wire x1="18.05" y1="16.5" x2="12.4239" y2="15.123878125" width="4" layer="1"/>
 <wire x1="12.4239" y1="15.123878125" x2="10.38811875" y2="14.498" width="4" layer="1"/>
 <wire x1="10.38811875" y1="14.498" x2="4.8" y2="12.78" width="4" layer="1"/>
@@
 <contactref element="U2" pad="5"/>
 <contactref element="R1" pad="V-"/>
-<wire x1="16.9" y1="20.06" x2="18.76" y2="20.06" width="0.4064" layer="1"/>
+<wire x1="18.05" y1="20.06" x2="18.76" y2="20.06" width="0.4064" layer="1"/>
 <wire x1="18.76" y1="20.06" x2="20" y2="21.3" width="0.4064" layer="1"/>
 <wire x1="20" y1="21.3" x2="20" y2="22.3274" width="0.4064" layer="1"/>
