File: Eagle_files/Final Project Designs_v1.brd (EAGLE design)
At the start: 100 x 80 mm, 29 parts, among them CON1 header, CON2 4PIN_GROVE_CONNECTORUNIVERSAL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, U1 TPS63000DRCR, U2 ATXMEGA32AA, X1 USB-MICROB", X4 JTAG, X5 BANANA_PLUG, X6 BANANA_PLUG

Commit message: added some files
Parts:
- moved F1 1.71 mm to (31.5, 15.2)
- moved R7 0.20 mm to (35.9, 31.7)
Routing:
- net N$16: track 5.31 -> 8.25 mm
- net N$23: track 34.1 -> 35.1 mm
Other:
- board text added: "Design by Rajith Radhakrishnan"
- board text added: "Thanks frank for the usb idea"

Commit message: added few more files
Routing:
- net N$16: track 8.25 -> 6.37 mm
- net N$15: track 4.70 -> 3.55 mm
- net N$23: track 35.1 -> 34.3 mm
Other:
- board text added: "Current Meter design"
- board text added: "ESE 323 design"
- board text added: "Thanks frank yee for usb idea, and taking the responsibility for ordering parts, pcb and taking in charge."
- board text added: "Touch to see effects of darwinism"
- board text added: "rated for 7A max"
- board text added: "special thanks to Prof. Westerfeld, Jeremiah, Frank Yee Juan for design suggestions, ideas and keeping my stupidity in check"

Commit message: update design and files
Routing:
- net N$6: track 24.8 -> 26.7 mm
Changed lines of the file:
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@@
 <contactref element="X3" pad="4"/>
 <contactref element="X1" pad="GND"/>
-<wire x1="20.01" y1="9.12" x2="25.33" y2="3.8" width="0.4064" layer="16"/>
-<wire x1="25.33" y1="3.8" x2="35.8" y2="3.8" width="0.4064" layer="16"/>
+<wire x1="20.01" y1="9.12" x2="21.43" y2="3.8" width="0.4064" layer="16"/>
+<wire x1="21.43" y1="3.8" x2="35.8" y2="3.8" width="0.4064" layer="16"/>
 <wire x1="35.8" y1="3.8" x2="35.8" y2="6" width="0.4064" layer="16"/>
 <via x="35.8" y="6" extent="1-16" drill="0.6" shape="octagon"/>
@@
 <wire x1="4.8" y1="12.78" x2="11.921553125" y2="14.779409375" width="4" layer="1"/>
 <wire x1="11.921553125" y1="14.779409375" x2="12.32975625" y2="14.894015625" width="4" layer="1"/>
-<wire x1="13.01" y1="9.12" x2="12.32975625" y2="14.894015625" width="1.27" layer="1"/>
+<wire x1="13.01" y1="9.12" x2="12.32975625" y2="14.894015625" width="0.6096" layer="1"/>
 <wire x1="17.1" y1="16.5" x2="11.921553125" y2="14.779409375" width="4" layer="1"/>
 </signal>
@@
 <wire x1="40.1" y1="13.58" x2="37.790196875" y2="14.485284375" width="4" layer="1"/>
 <wire x1="37.790196875" y1="14.485284375" x2="32.96" y2="16.09" width="4" layer="1"/>
-<wire x1="29.64" y1="5.205" x2="29.64" y2="5.86" width="0.4064" layer="1"/>
-<wire x1="29.64" y1="5.86" x2="27.8" y2="7.7" width="0.6096" layer="1"/>
 <wire x1="27.8" y1="7.7" x2="27.8" y2="8.5" width="0.6096" layer="1"/>
 <wire x1="27.8" y1="8.5" x2="29" y2="9.7" width="0.6096" layer="1"/>
@@
 <wire x1="36.8" y1="13.7" x2="37.0049125" y2="13.7" width="0.4064" layer="1"/>
 <wire x1="37.0049125" y1="13.7" x2="37.790196875" y2="14.485284375" width="0.4064" layer="1"/>
+<wire x1="29.64" y1="5.86" x2="27.8" y2="7.7" width="0.6096" layer="1"/>
+<wire x1="29.64" y1="5.205" x2="29.64" y2="5.86" width="0.6096" layer="1"/>
 </signal>
 <signal name="N$15">

Commit message: finished everthing
Parts:
- removed GND-, VIN+: TP-1502, sps:TP-1502
- added U$1: BATTERY, Tft_lcd_header:BATTERY
- moved PB2 2.43 mm to (29.2, 45.5)
- moved PB1 1.32 mm to (18.8, 45.9)
- moved X5 1.24 mm to (4.41, 8.88)
- moved R4 0.32 mm to (37.4, 24.1)
- moved R6 0.32 mm to (36.6, 29.2)
- moved COUT_1 0.32 mm to (6.99, 21.7)
- moved COUT_2 0.32 mm to (10.5, 21.7)
- moved F1 0.32 mm to (31.6, 15.5)
- moved R1 0.32 mm to (20.2, 19.5)
- moved R2 0.32 mm to (31.3, 20.7)
- moved R9 0.32 mm to (25.8, 39.1)
- moved RFBB 0.32 mm to (6.09, 30.1)
- moved RFBT 0.32 mm to (9.68, 30.1)
- moved U1 0.32 mm to (8.94, 26.4)
- moved U2 0.32 mm to (19.8, 26.9)
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Connections:
- net GND: now also U$1.GND; no longer GND-.1
- net VIN: now also U$1.VCC; no longer VIN+.1
Routing:
- net +3V3: track 126.4 -> 125.3 mm
- net VIN: track 37.4 -> 38.4 mm
- net B$2: track 29.3 -> 30.3 mm
- net N$10: track 22.6 -> 23.3 mm
Other:
- board size 100 x 80 mm -> 52.9 x 52.6 mm
- board text added: "https://radrajith.github.io/ESE_323_PCB_Design/"
- board text removed: "Thanks frank yee for usb idea, and taking the responsibility for ordering parts, pcb and taking in charge."
