File: TPS63000/Eagle/SPS/2016-10-14_05-18-27.sch (EAGLE design)
At the start: 19 parts, among them IC1 ATXMEGA32AA, J1 USB-MICROB", U1 TPS63000DRCR

Commit message: updated designs
Parts:
- removed IC1: ATXMEGA32AA, Tft_lcd_header:ATXMEGA32AA
- removed J1: USB-MICROB", SparkFun-Connectors:USB-MICROB"
- removed SV1: (no value), Tft_lcd_header:14_PIN_FEMALE_HEADER
- removed SW1, SW2: (no value), buttons:10-XX-4.5SMD
- removed U$1: 4PIN_GROVE_CONNECTORUNIVERSAL_4_PIN_CONNECTOR, Tft_lcd_header:4PIN_GROVE_CONNECTORUNIVERSAL_4_PIN_CONNECTOR
- removed U$2: RESISTOR_4PIN, Tft_lcd_header:RESISTOR_4PIN
- removed X1: (no value), con-berg:PN87520
Connections:
- removed net +3V3: IC1.AVCC, IC1.VCC, SV1.LED, SV1.VCC, SW1.P1, SW2.P1, U$1.VCC
- removed net GND1: COUT_1.2, COUT_2.2, GND.1@1, GND1.TP, RFBB.2@2, U1.GND@9, U1.PAD@11, U1.PGND@3, VIN.-@2
- removed net N$1: IC1.(MOSI)PC7, SV1.MOSI
- removed net N$10: IC1.(RXD)PD0, SW1.S1
- removed net N$11: U$1.GND
- removed net N$12: J1.VBUS, U$2.I_IN
- removed net N$13: U$2.I_OUT, X1.1
- removed net N$14: IC1.PA0(ADC0)
- removed net N$15: IC1.PA1(ADC1), U$2.V-
- removed net N$2: SV1.SCK
- removed net N$3: IC1.(MISO)PC6, SV1.MISO
- removed net N$4: IC1.(SCL)PC1, U$1.SCL
- removed net N$5: U$1.SDA
- removed net N$6: X1.4
- removed net N$7: J1.D+, X1.2
- removed net N$8: J1.D-, X1.3
- removed net N$9: IC1.(TXD)PD1, SW2.S1
- net GND: now also CIN.1, COUT_1.2, COUT_2.2, GND.1@1, GND1.TP, RFBB.2@2, U1.GND@9, U1.PAD@11, U1.PGND@3, VIN.-@2; no longer IC1.GND, SV1.GND
