File: TPS63000/Eagle/sps/2016-10-14_05-17-29.sch (EAGLE design)
At the start: 11 parts, among them U1 TPS63000DRCR

Commit message: updated designs, downloaded some datasheets, modified the BOM
Parts:
- removed GND1, VOUT: TP-1502, sps:TP-1502
- added RLOAD: WB_LOAD_RESISTOR, AcceleratedDesigns_Lib:WB_LOAD_RESISTORWB_LOAD_RESISTOR
- renumbered COUT_1 to COUT
Connections:
- removed net GND1: CIN.2@2, COUT.2@2, COUT_2.2@2, GND.1@1, GND1.TP, U1.GND@9, U1.PAD@11, U1.PGND@3, VIN.-@2
- removed net N$1: RFBT.1@1
- removed net N$2: RFBB.2@2
- removed net VOUT: COUT.1@1, COUT_2.1@1, U1.VOUT@1, VOUT.TP
- new net 0: CIN.2@2, COUT.2@2, COUT_2.2@2, GND.1@1, RFBB.2@2, RLOAD.2@2, U1.GND@9, U1.PAD@11, U1.PGND@3, VIN.-@2
- new net 6: COUT.1@1, COUT_2.1@1, RFBT.1@1, RLOAD.1@1, U1.VOUT@1
Changed lines of the file:
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@@
 <setting verticaltext="up"/>
 </settings>
-<grid distance="0.1" unitdist="inch" unit="inch" style="lines" multiple="1" display="no" altdistance="0.01" altunitdist="inch" altunit="inch"/>
+<grid distance="0.1" unitdist="inch" unit="mil" style="lines" multiple="1" display="no" altdistance="0.01" altunitdist="inch" altunit="inch"/>
 <layers>
-<layer number="1" name="Top" color="4" fill="1" visible="no" active="no"/>
-<layer number="16" name="Bottom" color="1" fill="1" visible="no" active="no"/>
-<layer number="17" name="Pads" color="2" fill="1" visible="no" active="no"/>
-<layer number="18" name="Vias" color="2" fill="1" visible="no" active="no"/>
-<layer number="19" name="Unrouted" color="6" fill="1" visible="no" active="no"/>
-<layer number="20" name="Dimension" color="15" fill="1" visible="no" active="no"/>
-<layer number="21" name="tPlace" color="7" fill="1" visible="no" active="no"/>
-<layer number="22" name="bPlace" color="7" fill="1" visible="no" active="no"/>
-<layer number="23" name="tOrigins" color="15" fill="1" visible="no" active="no"/>
-<layer number="24" name="bOrigins" color="15" fill="1" visible="no" active="no"/>
-<layer number="25" name="tNames" color="7" fill="1" visible="no" active="no"/>
-<layer number="26" name="bNames" color="7" fill="1" visible="no" active="no"/>
-<layer number="27" name="tValues" color="7" fill="1" visible="no" active="no"/>
-<layer number="28" name="bValues" color="7" fill="1" visible="no" active="no"/>
-<layer number="29" name="tStop" color="7" fill="3" visible="no" active="no"/>
-<layer number="30" name="bStop" color="7" fill="6" visible="no" active="no"/>
-<layer number="31" name="tCream" color="7" fill="4" visible="no" active="no"/>
-<layer number="32" name="bCream" color="7" fill="5" visible="no" active="no"/>
-<layer number="33" name="tFinish" color="6" fill="3" visible="no" active="no"/>
-<layer number="34" name="bFinish" color="6" fill="6" visible="no" active="no"/>
-<layer number="35" name="tGlue" color="7" fill="4" visible="no" active="no"/>
-<layer number="36" name="bGlue" color="7" fill="5" visible="no" active="no"/>
-<layer number="37" name="tTest" color="7" fill="1" visible="no" active="no"/>
-<layer number="38" name="bTest" color="7" fill="1" visible="no" active="no"/>
-<layer number="39" name="tKeepout" color="4" fill="11" visible="no" active="no"/>
-<layer number="40" name="bKeepout" color="1" fill="11" visible="no" active="no"/>
-<layer number="41" name="tRestrict" color="4" fill="10" visible="no" active="no"/>
-<layer number="42" name="bRestrict" color="1" fill="10" visible="no" active="no"/>
-<layer number="43" name="vRestrict" color="2" fill="10" visible="no" active="no"/>
-<layer number="44" name="Drills" color="7" fill="1" visible="no" active="no"/>
-<layer number="45" name="Holes" color="7" fill="1" visible="no" active="no"/>
-<layer number="46" name="Milling" color="3" fill="1" visible="no" active="no"/>
-<layer number="47" name="Measures" color="7" fill="1" visible="no" active="no"/>
-<layer number="48" name="Document" color="7" fill="1" visible="no" active="no"/>
-<layer number="49" name="Reference" color="7" fill="1" visible="no" active="no"/>
-<layer number="51" name="tDocu" color="7" fill="1" visible="no" active="no"/>
-<layer number="52" name="bDocu" color="7" fill="1" visible="no" active="no"/>
-<layer number="90" name="Modules" color="5" fill="1" visible="yes" active="yes"/>
 <layer number="91" name="Nets" color="2" fill="1" visible="yes" active="yes"/>
 <layer number="92" name="Busses" color="1" fill="1" visible="yes" active="yes"/>
@@
 <parts>
 <part name="CIN" library="AcceleratedDesigns_Lib" deviceset="LMK212BJ106KG-T" device="LMK212BJ106KG-T" value="10uF"/>
-<part name="COUT_1" library="AcceleratedDesigns_Lib" deviceset="LMK212BJ226MG-T" device="LMK212BJ226MG-T" value="22uF"/>
+<part name="COUT" library="AcceleratedDesigns_Lib" deviceset="LMK212BJ226MG-T" device="LMK212BJ226MG-T" value="22uF"/>
 <part name="GND" library="AcceleratedDesigns_Lib" deviceset="WB_GND" device="WB_GND" value="WB_GND"/>
 <part name="L1" library="AcceleratedDesigns_Lib" deviceset="LQM21PN1R5MC0D" device="LQM21PN1R5MC0D" value="1.5uH"/>
@@
 <part name="U1" library="AcceleratedDesigns_Lib" deviceset="TPS63000DRCR" device="TPS63000DRCR" value="TPS63000DRCR"/>
 <part name="VIN" library="AcceleratedDesigns_Lib" deviceset="WB_STARTUP_VOLTAGE_SOURCE" device="WB_STARTUP_VOLTAGE_SOURCE" value="WB_STARTUP_VOLTAGE_SOURCE"/>
+<part name="RLOAD" library="AcceleratedDesigns_Lib" deviceset="WB_LOAD_RESISTOR" device="WB_LOAD_RESISTOR" value="WB_LOAD_RESISTOR"/>
 <part name="COUT_2" library="AcceleratedDesigns_Lib" deviceset="LMK212BJ226MG-T" device="LMK212BJ226MG-T" value="22uF"/>
-<part name="VOUT" library="sps" deviceset="TP-1502" device=""/>
-<part name="GND1" library="sps" deviceset="TP-1502" device=""/>
 </parts>
 <sheets>
@@
 <attribute name="VALUE" x="51.308" y="61.976" size="2" layer="96"/>
 </instance>
-<instance part="COUT_1" gate="1" x="149.86" y="63.5" smashed="yes" rot="R90">
+<instance part="COUT" gate="1" x="149.86" y="63.5" smashed="yes" rot="R90">
 <attribute name="NAME" x="152.908" y="67.818" size="2" layer="95"/>
 <attribute name="VALUE" x="152.908" y="63.246" size="2" layer="96"/>
@@
 <attribute name="NAME" x="35.052" y="71.882" size="2" layer="95"/>
 </instance>
+<instance part="RLOAD" gate="1" x="190.5" y="48.26" smashed="yes" rot="R90">
+<attribute name="NAME" x="192.024" y="51.054" size="2" layer="95"/>
+</instance>
 <instance part="COUT_2" gate="1" x="167.64" y="63.5" smashed="yes" rot="R90">
 <attribute name="NAME" x="170.688" y="67.818" size="2" layer="95"/>
 <attribute name="VALUE" x="170.688" y="63.246" size="2" layer="96"/>
 </instance>
-<instance part="VOUT" gate="A" x="190.5" y="86.36" rot="R180"/>
-<instance part="GND1" gate="A" x="190.5" y="30.48" rot="R180"/>
 </instances>
 <busses>
@@
 </segment>
 </net>
-<net name="GND1" class="0">
-<segment>
-<pinref part="U1" gate="1" pin="GND@9"/>
-<wire x1="109.22" y1="66.04" x2="109.22" y2="30.48" width="0" layer="91"/>
-</segment>
+<net name="0" class="0">
 <segment>
 <pinref part="CIN" gate="1" pin="2@2"/>
-<wire x1="48.26" y1="54.61" x2="48.26" y2="30.48" width="0" layer="91"/>
-</segment>
-<segment>
-<pinref part="COUT_2" gate="1" pin="2@2"/>
-<pinref part="COUT_1" gate="1" pin="2@2"/>
-<wire x1="149.86" y1="55.88" x2="167.64" y2="55.88" width="0" layer="91"/>
-<wire x1="149.86" y1="55.88" x2="149.86" y2="30.48" width="0" layer="91"/>
-</segment>
-<segment>
+<pinref part="COUT" gate="1" pin="2@2"/>
 <pinref part="GND" gate="1" pin="1@1"/>
+<pinref part="RFBB" gate="1" pin="2@2"/>
 <pinref part="U1" gate="1" pin="PGND@3"/>
+<pinref part="U1" gate="1" pin="GND@9"/>
 <pinref part="U1" gate="1" pin="PAD@11"/>
 <pinref part="VIN" gate="1" pin="-@2"/>
+<pinref part="RLOAD" gate="1" pin="2@2"/>
+<pinref part="COUT_2" gate="1" pin="2@2"/>
+<wire x1="48.26" y1="54.61" x2="48.26" y2="30.48" width="0" layer="91"/>
+<wire x1="109.22" y1="66.04" x2="109.22" y2="30.48" width="0" layer="91"/>
+<wire x1="127" y1="35.56" x2="127" y2="30.48" width="0" layer="91"/>
+<wire x1="149.86" y1="55.88" x2="149.86" y2="30.48" width="0" layer="91"/>
 <wire x1="30.48" y1="30.48" x2="190.5" y2="30.48" width="0" layer="91"/>
 <wire x1="30.48" y1="30.48" x2="30.48" y2="58.42" width="0" layer="91"/>
-<label x="165.1" y="25.4" size="1.778" layer="95"/>
-<pinref part="GND1" gate="A" pin="TP"/>
+<wire x1="190.5" y1="30.48" x2="190.5" y2="40.64" width="0" layer="91"/>
+<wire x1="149.86" y1="55.88" x2="167.64" y2="55.88" width="0" layer="91"/>
 </segment>
 </net>
-<net name="VOUT" class="0">
+<net name="6" class="0">
 <segment>
+<pinref part="COUT" gate="1" pin="1@1"/>
+<pinref part="RFBT" gate="1" pin="1@1"/>
+<pinref part="U1" gate="1" pin="VOUT@1"/>
+<pinref part="RLOAD" gate="1" pin="1@1"/>
 <pinref part="COUT_2" gate="1" pin="1@1"/>
-<pinref part="COUT_1" gate="1" pin="1@1"/>
+<wire x1="127" y1="83.82" x2="127" y2="86.36" width="0" layer="91"/>
 <wire x1="149.86" y1="71.12" x2="149.86" y2="86.36" width="0" layer="91"/>
+<wire x1="109.22" y1="86.36" x2="190.5" y2="86.36" width="0" layer="91"/>
+<wire x1="190.5" y1="55.88" x2="190.5" y2="86.36" width="0" layer="91"/>
 <wire x1="149.86" y1="71.12" x2="167.64" y2="71.12" width="0" layer="91"/>
-</segment>
-<segment>
-<pinref part="U1" gate="1" pin="VOUT@1"/>
-<wire x1="109.22" y1="86.36" x2="190.5" y2="86.36" width="0" layer="91"/>
-<label x="162.56" y="88.9" size="1.778" layer="95"/>
-<pinref part="VOUT" gate="A" pin="TP"/>
 </segment>
 </net>
@@
 </segment>
 </net>
-<net name="N$1" class="0">
-<segment>
-<pinref part="RFBT" gate="1" pin="1@1"/>
-<wire x1="127" y1="83.82" x2="127" y2="86.36" width="0" layer="91"/>
-</segment>
-</net>
-<net name="N$2" class="0">
-<segment>
-<pinref part="RFBB" gate="1" pin="2@2"/>
-<wire x1="127" y1="35.56" x2="127" y2="30.48" width="0" layer="91"/>
-</segment>
-</net>
